File: KiCAD/ddc112-shield/LED_driver.kicad_sch (KiCad schematic)
At the start: 12 parts, among them Q1 TTC1949, U7 TLV272IS-13, U8 MCP4922-EP

Commit message: woring on LED driver
Parts:
- removed U8: MCP4922-EP, Package_SO:SOIC-14_3.9x8.7mm_P1.27mm, symbol Analog_DAC:MCP4922-EP
- added C15: 0.33uF, Capacitor_SMD:C_0603_1608Metric, symbol Device:C_Small
- added C16: 0.1uF, Capacitor_SMD:C_0603_1608Metric, symbol Device:C_Small
- added Q2, Q3, Q4: TTC1949, Package_TO_SOT_SMD:SC-59, symbol Device:Q_NPN_BEC
- added U6: LTC1380, symbol my_LTC1380:LTC1380
- added U9: LTC2631, Package_TO_SOT_SMD:TSOT-23-8, symbol my_LTC2631:LTC2631
- C21: value 0.1uF -> 1nF
- C22: footprint Capacitor_SMD:C_0805_2012Metric_Pad1.18x1.45mm_HandSolder -> Capacitor_SMD:C_0603_1608Metric; DigikeyNumber (none) -> 1276-1005-1-ND; ManufacturerNumber (none) -> CL10B104KO8NNNC
- R4: value 1k -> 440
Connections:
- net Earth: now also U6.1 (0), U6.10 (VEE)
- net GND: now also C15.2, C16.2, U6.12 (A1), U6.13 (A0), U9.1 (CA0), U9.4 (GND)
- net LED_PWR_5V: now also Q1.1 (B), C16.1, Q2.1 (B), Q2.3 (C), Q3.1 (B), Q3.3 (C), Q4.3 (C), U6.1 (0), U6.16 (VCC), U6.2 (1), U6.3 (2), U9.5 (VCC), U9.8 (REF_SEL)
- net at R5.1: now also U6.9 (I/O); no longer Q1.1 (B)
- net at R3.2: now also U9.7 (Vout)
- net LED_A renamed LED_1
- new net: Q4.1 (B), U6.4 (3)
- new net: C15.1, U9.6 (REF)
- new net LED_2: Q2.2 (E)
- new net LED_3: Q3.2 (E)
- new net LED_4: Q4.2 (E)
- new net SCL: U6.15 (SCL), U9.2 (SCL)
- new net SDA: U6.14 (SDA), U9.3 (SDA)
Other:
- note added: "1.25V @ 50mA"
- note added: "170mV"
- note added: "DAC range 0...4.095V"
- note added: "LED drive 0-1.25V for 0-50mA"
- note added: "V(BE) ~ 200mV"
- note added: "V(F) = 2V @ 50mA"
- note added: "hFE = 300 @ 50mA"
- note removed: "DAC out 0-2.5 or 0-5V"
- note removed: "LED drive 0-1.25V"
- moved on the sheet: Q1, R6, R7

Commit message: LED driver schematic complete?
Parts:
- removed U7: TLV272IS-13, Package_SO:SOIC-8_3.9x4.9mm_P1.27mm, symbol TLV272IS-13:TLV272IS-13
- added U8: OPA365xxD, Package_SO:SOIC-8_3.9x4.9mm_P1.27mm, symbol Amplifier_Operational:OPA365xxD
- C15, C16, C22: footprint Capacitor_SMD:C_0603_1608Metric -> Capacitor_SMD:C_0805_2012Metric_Pad1.18x1.45mm_HandSolder
- U6: footprint (none) -> Package_SO:SOIC-16_3.9x9.9mm_P1.27mm; DigikeyNumber (none) -> 505-LTC1380CS#PBF-ND
Connections:
- net Earth: now also C22.2, U6.12 (A1), U6.13 (A0), U8.4 (V-)
- net GND: no longer C22.2, U6.12 (A1), U6.13 (A0)
- net LED_PWR_5V: now also U8.7 (V+)
- net at C17.1, R6.2: now also U8.2 (-)
- net at C17.2, R5.2: now also U8.6
- net at C21.1, R3.1, R4.1: now also U8.3 (+)
Other:
- note removed: "1.25V @ 50mA"
- moved on the sheet: C15, C16, C17, C21, C22, R3, R4, R6, R7, U9
