File: KiCAD/led-photodiode-avr/led-photodiode-avr.kicad_pcb (KiCad board)
At the start: 4 copper layers, 68.6 x 80 mm, 58 parts, among them J1 Screw_Terminal_01x02, J2 Conn_02x08_Odd_Even, J3 ISP, J4 Conn_01x06_Pin, Q1 TTC1949, Q2 TTC1949, Q3 TTC1949, Q4 TTC1949, U1 REF3040, U2 L78L05_SOT89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

Commit message: many schematic tweaks; add fields for BOM
Parts:
- removed U4: L78L05_SOT89, Package_TO_SOT_SMD:SOT-89-3
- added D1: LED, LED_SMD:LED_0805_2012Metric_Pad1.15x1.40mm_HandSolder, F.Cu at (208.9, 73.3)
- added D2: LED, LED_SMD:LED_0805_2012Metric_Pad1.15x1.40mm_HandSolder, F.Cu at (208.9, 76.3)
- added L1: 10uH, Inductor_SMD:L_0805_2012Metric_Pad1.15x1.40mm_HandSolder, F.Cu at (217.9, 91.7)
- added R10: 1.5k, Resistor_SMD:R_0805_2012Metric_Pad1.20x1.40mm_HandSolder, F.Cu at (213.6, 76.2)
- added U10: AZ1117CH2-5.0, Package_TO_SOT_SMD:SOT-223-3_TabPin2, F.Cu at (210.6, 96.2)
- C1: value 0.47uF -> 0.33uF
- C2, C7: value 0.33uF -> 10uF
- C3, C8: value 0.1uF -> 22uF
- L2: footprint Inductor_SMD:L_0603_1608Metric_Pad1.05x0.95mm_HandSolder -> Inductor_SMD:L_0805_2012Metric_Pad1.15x1.40mm_HandSolder
- R2: value 0R -> 1.5k
- R4: value 440 -> 442
- R7: value 25 -> 24.9
- U1: value REF3040 -> REF3040AIDBZT
- U2: value L78L05_SOT89 -> AZ1117CH2-5.0; footprint Package_TO_SOT_SMD:SOT-89-3 -> Package_TO_SOT_SMD:SOT-223-3_TabPin2
- U3: value OPA350 -> OPA365xxD
- moved R2 65.1 mm to (213.6, 73.2)
- moved U3 56.1 mm to (219.8, 87.0), turned to 0 degrees
- moved U2 54.1 mm to (210.6, 87.8)
Connections:
- R2 pad 1: GND -> +5VA
- R2 pad 2: Earth -> Net-(D1-A)
- U2 pad 1: +5VA -> VBUS
- U2 pad 2: Earth -> GND
- U2 pad 3: VBUS -> VCC
- U3 pad 1: /VREF -> unconnected-(U3-NC-Pad1)
- U3 pad 5: (no net) -> unconnected-(U3-NC-Pad5)
- U3 pad 6: (no net) -> /VREF
- U3 pad 7: (no net) -> +5VA
- U3 pad 8: +5VA -> unconnected-(U3-NC-Pad8)

Commit message: routing done
Parts:
- added H1: MountingHole, MountingHole:MountingHole_4.3mm_M4_DIN965_Pad, F.Cu at (121.9, 62.2)
- added H2: MountingHole, MountingHole:MountingHole_4.3mm_M4_DIN965_Pad, F.Cu at (180.3, 62.2)
- added H3: MountingHole, MountingHole:MountingHole_4.3mm_M4_DIN965_Pad, F.Cu at (121.9, 132.1)
- added H4: MountingHole, MountingHole:MountingHole_4.3mm_M4_DIN965_Pad, F.Cu at (180.3, 132.1)
- moved R10 84.9 mm to (147.3, 129.3), turned to 90 degrees
- moved D2 84.4 mm to (147.3, 134.0), turned to 90 degrees
- moved U2 84.1 mm to (139.1, 132.1)
- moved D1 70.6 mm to (172.7, 134.0), turned to 90 degrees
- moved R2 69.4 mm to (172.7, 129.2), turned to 90 degrees
- moved L1 64.1 mm to (154.9, 103.5)
- moved U10 57.6 mm to (165.7, 132.3)
- moved U3 54.1 mm to (172.7, 113.7)
- moved C8 31.9 mm to (130.8, 134.6)
- moved R29 31.0 mm to (130.0, 94.2), turned to 180 degrees
- moved J1 27.0 mm to (120.6, 117.8)
- moved C7 24.2 mm to (130.8, 129.5)
- moved J4 24.2 mm to (124.5, 100.3)
- moved J3 18.2 mm to (122.6, 78.7), turned to 180 degrees
- moved R45 18.2 mm to (132.1, 77.5)
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Connections:
- C16 pad 1: +5VA -> VCC
- D1 pad 1: GND -> Earth
- J2 pad 1: /LED_driver/LED_1 -> /LED_driver/LED_3
- J2 pad 9: /LED_driver/LED_3 -> /LED_driver/LED_1
- U6 pad 11: Earth -> GND
- U6 pad 12: Earth -> GND
- U6 pad 13: Earth -> GND
- U9 pad 5: +5VA -> VCC
- U9 pad 8: +5VA -> VCC
Routing:
- net /MOSI: track 0.00 -> 67.1 mm, vias 0 -> 3
- net /SCK: track 0.00 -> 63.7 mm, vias 0 -> 3
- net /MISO: track 0.00 -> 63.5 mm, vias 0 -> 2
- net VBUS: track 0.00 -> 57.6 mm
- net /PC2/ADC2: track 0.00 -> 52.0 mm
- net GND: track 0.00 -> 42.5 mm, vias 0 -> 23
- net Earth: track 0.00 -> 41.7 mm, vias 0 -> 22
- net /PC1/ADC1: track 0.00 -> 40.4 mm
- net /PC0/ADC0: track 0.00 -> 38.9 mm
- net /PD7: track 0.00 -> 38.5 mm, vias 0 -> 2
- net /SCL: track 0.00 -> 38.3 mm, vias 0 -> 2
- net /PD5: track 0.00 -> 34.7 mm, vias 0 -> 2
- net VCC: track 0.00 -> 32.3 mm, vias 0 -> 15
- net /PD6/OC0A: track 0.00 -> 31.5 mm, vias 0 -> 2
- net /SDA: track 0.00 -> 30.6 mm
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- added copper zone on In2.Cu, net +5VA
- added copper zone on B.Cu, net Earth
- added copper zone on F.Cu, net Earth
- added copper zone on In2.Cu, net VCC
Other:
- board text added: "+9V"
- board text added: "1"
- board text added: "G"
- board text added: "GND"
- board text added: "ISP 5V"
- board text added: "RX"
- board text added: "SWIR Wearable Optical Test V1.0 -2025-08 E. Hazen"
- board text added: "TX"

Commit message: ready for review
Parts:
- J1: footprint TerminalBlock:TerminalBlock_MaiXu_MX126-5.0-02P_1x02_P5.00mm -> my_ScrewTerminal:TerminalBlock_TE_2POS_P5mm
Routing:
- net VBUS: track 57.6 -> 66.0 mm
- added copper zone on F.Cu, net GND
Other:
- board text removed: "G"

Commit message: small tweaks
Parts:
- J3: footprint Connector_PinHeader_2.54mm:PinHeader_2x03_P2.54mm_Vertical -> Connector_IDC:IDC-Header_2x03_P2.54mm_Horizontal
- U8: value OPA365xxD -> OPA365AIDR
Other:
- board text added: "NIR Wearable Optical Test V1.0 -2025-08 E. Hazen"
- board text removed: "SWIR Wearable Optical Test V1.0 -2025-08 E. Hazen"
Changed lines of the file:
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@@
 		)
 		(embedded_fonts no)
-		(model "${KICAD9_3DMODEL_DIR}/TerminalBlock.3dshapes/TerminalBlock_MaiXu_MX126-5.0-02P_1x02_P5.00mm.step"
+		(model "${KIPRJMOD}/models/282836-2.step"
 			(offset
-				(xyz 0 0 0)
+				(xyz 2.5 4 5)
 			)
 			(scale
@@
 			)
 			(rotate
-				(xyz 0 0 0)
+				(xyz -90 -0 -180)
 			)
 		)
@@
 		)
 	)
-	(footprint "Connector_PinHeader_2.54mm:PinHeader_2x03_P2.54mm_Vertical"
+	(footprint "Connector_IDC:IDC-Header_2x03_P2.54mm_Horizontal"
 		(layer "F.Cu")
 		(at 122.56 78.74 180)
-		(descr "Through hole straight pin header, 2x03, 2.54mm pitch, double rows")
-		(tags "Through hole pin header THT 2x03 2.54mm double row")
+		(descr "Through hole IDC box header, 2x03, 2.54mm pitch, DIN 41651 / IEC 60603-13, double rows, https://docs.google.com/spreadsheets/d/16SsEcesNF15N3Lb4niX7dcUr-NY5_MFPQhobNuNppn4/edit#gid=0")
+		(tags "Through hole horizontal IDC box header THT 2x03 2.54mm double row")
 		(property "Reference" "J3"
-			(at 3.92 -3.81 0)
+			(at 6.215 -6.1 180)
 			(layer "F.SilkS")
 			(effects
 				(font
-					(size 1.524 1.524)
-					(thickness 0.1778)
+					(size 1 1)
+					(thickness 0.15)
 				)
 			)
 		)
 		(property "Value" "ISP"
-			(at 1.27 7.46 0)
+			(at 6.215 11.18 180)
 			(layer "F.Fab")
 			(effects
@@
 			)
 		)
-		(property "Datasheet" "~"
-			(at 0 0 0)
+		(property "Datasheet" "https://media.metz-connect.com/files/171/Data_sheet_PR202XXVBDN.PDF"
+			(at 0 0 180)
 			(layer "F.Fab")
 			(hide yes)
@@
 		)
 		(property "Description" ""
-			(at 0 0 0)
+			(at 0 0 180)
 			(layer "F.Fab")
 			(hide yes)
@@
 			)
 		)
-		(property "DigikeyNumber" "1849-PR20203VBDN-ND"
+		(property "DigikeyNumber" "952-2092-ND"
 			(at 0 0 180)
 			(unlocked yes)
@@
 			)
 		)
-		(property "ManufacturerNumber" "PR20203VBDN"
+		(property "ManufacturerNumber" "M20-9950345"
 			(at 0 0 180)
 			(unlocked yes)
@@
 		(attr through_hole)
 		(fp_line
-			(start 3.92 -1.38)
-			(end 3.92 6.46)
+			(start 13.39 10.29)
+			(end 4.27 10.29)
 			(stroke
 				(width 0.12)
@@
 		)
 		(fp_line
-			(start 1.27 1.27)
-			(end 1.27 -1.38)
+			(start 13.39 -5.21)
+			(end 13.39 10.29)
 			(stroke
 				(width 0.12)
@@
 		)
 		(fp_line
-			(start 1.27 -1.38)
-			(end 3.92 -1.38)
+			(start 4.27 10.29)
+			(end 4.27 -5.21)
 			(stroke
 				(width 0.12)
@@
 		)
 		(fp_line
-			(start -1.38 6.46)
-			(end 3.92 6.46)
+			(start 4.27 4.59)
+			(end 13.39 4.59)
 			(stroke
 				(width 0.12)
@@
 		)
 		(fp_line
-			(start -1.38 1.27)
-			(end 1.27 1.27)
+			(start 4.27 0.49)
+			(end 13.39 0.49)
 			(stroke
 				(width 0.12)
@@
 		)
 		(fp_line
-			(start -1.38 1.27)
-			(end -1.38 6.46)
+			(start 4.27 -5.21)
+			(end 13.39 -5.21)
 			(stroke
 				(width 0.12)
@@
 		)
 		(fp_line
-			(start -1.38 0)
-			(end -1.38 -1.38)
+			(start -1.35 0)
+			(end -2.35 -0.5)
 			(stroke
 				(width 0.12)
@@
 		)
 		(fp_line
-			(start -1.38 -1.38)
-			(end 0 -1.38)
+			(start -2.35 0.5)
+			(end -1.35 0)
 			(stroke
 				(width 0.12)
@@
 		)
 		(fp_line
-			(start 4.32 6.85)
-			(end 4.32 -1.77)
+			(start -2.35 -0.5)
+			(end -2.35 0.5)
+			(stroke
+				(width 0.12)
+				(type solid)
+			)
+			(layer "F.SilkS")
+		)
+		(fp_line
+			(start 13.78 10.69)
+			(end 13.78 -5.6)
 			(stroke
 				(width 0.05)
@@
 		)
 		(fp_line
-			(start 4.32 -1.77)
-			(end -1.77 -1.77)
+			(start 13.78 -5.6)
+			(end -1.35 -5.6)
 			(stroke
 				(width 0.05)
@@
 		)
 		(fp_line
-			(start -1.77 6.85)
-			(end 4.32 6.85)
+			(start -1.35 10.69)
+			(end 13.78 10.69)
 			(stroke
 				(width 0.05)
@@
 		)
 		(fp_line
-			(start -1.77 -1.77)
-			(end -1.77 6.85)
+			(start -1.35 -5.6)
+			(end -1.35 10.69)
 			(stroke
 				(width 0.05)
@@
 		)
 		(fp_line
-			(start 3.81 6.35)
-			(end -1.27 6.35)
+			(start 13.28 10.18)
+			(end 4.38 10.18)
 			(stroke
 				(width 0.1)
@@
 		)
 		(fp_line
-			(start 3.81 -1.27)
-			(end 3.81 6.35)
+			(start 13.28 -5.1)
+			(end 13.28 10.18)
 			(stroke
 				(width 0.1)
@@
 		)
 		(fp_line
-			(start 0 -1.27)
-			(end 3.81 -1.27)
+			(start 5.38 -5.1)
+			(end 13.28 -5.1)
 			(stroke
 				(width 0.1)
@@
 		)
 		(fp_line
-			(start -1.27 6.35)
-			(end -1.27 0)
+			(start 4.38 10.18)
+			(end 4.38 -4.1)
 			(stroke
 				(width 0.1)
@@
 		)
 		(fp_line
-			(start -1.27 0)
-			(end 0 -1.27)
+			(start 4.38 4.76)
+			(end -0.32 4.76)
+			(stroke
+				(width 0.1)
+				(type solid)
+			)
+			(layer "F.Fab")
+		)
+		(fp_line
+			(start 4.38 4.59)
+			(end 13.28 4.59)
+			(stroke
+				(width 0.1)
+				(type solid)
+			)
+			(layer "F.Fab")
+		)
+		(fp_line
+			(start 4.38 2.22)
+			(end -0.32 2.22)
+			(stroke
+				(width 0.1)
+				(type solid)
+			)
+			(layer "F.Fab")
+		)
+		(fp_line
+			(start 4.38 0.49)
+			(end 13.28 0.49)
+			(stroke
+				(width 0.1)
+				(type solid)
+			)
+			(layer "F.Fab")
+		)
+		(fp_line
+			(start 4.38 -0.32)
+			(end -0.32 -0.32)
+			(stroke
+				(width 0.1)
+				(type solid)
+			)
+			(layer "F.Fab")
+		)
+		(fp_line
+			(start 4.38 -4.1)
+			(end 5.38 -5.1)
+			(stroke
+				(width 0.1)
+				(type solid)
+			)
+			(layer "F.Fab")
+		)
+		(fp_line
+			(start -0.32 5.4)
+			(end 4.38 5.4)
+			(stroke
+				(width 0.1)
+				(type solid)
+			)
+			(layer "F.Fab")
+		)
+		(fp_line
+			(start -0.32 4.76)
+			(end -0.32 5.4)
+			(stroke
+				(width 0.1)
+				(type solid)
+			)
+			(layer "F.Fab")
+		)
+		(fp_line
+			(start -0.32 2.86)
+			(end 4.38 2.86)
+			(stroke
+				(width 0.1)
+				(type solid)
+			)
+			(layer "F.Fab")
+		)
+		(fp_line
+			(start -0.32 2.22)
+			(end -0.32 2.86)
+			(stroke
+				(width 0.1)
+				(type solid)
+			)
+			(layer "F.Fab")
+		)
+		(fp_line
+			(start -0.32 0.32)
+			(end 4.38 0.32)
+			(stroke
+				(width 0.1)
+				(type solid)
+			)
+			(layer "F.Fab")
+		)
+		(fp_line
+			(start -0.32 -0.32)
+			(end -0.32 0.32)
 			(stroke
 				(width 0.1)
@@
 		)
 		(fp_text user "${REFERENCE}"
-			(at 1.27 2.54 90)
+			(at 8.83 2.54 270)
 			(layer "F.Fab")
 			(effects
 				(font
-					(size 1.524 1.524)
-					(thickness 0.1778)
+					(size 1 1)
+					(thickness 0.15)
 				)
 			)
 		)
-		(pad "1" thru_hole rect
+		(pad "1" thru_hole roundrect
 			(at 0 0 180)
 			(size 1.7 1.7)
@@
 			(layers "*.Cu" "*.Mask")
 			(remove_unused_layers no)
+			(roundrect_rratio 0.147059)
 			(net 31 "/MISO")
 			(pinfunction "MISO")
@@
 		)
 		(embedded_fonts no)
-		(model "${KICAD9_3DMODEL_DIR}/Connector_PinHeader_2.54mm.3dshapes/PinHeader_2x03_P2.54mm_Vertical.step"
+		(model "${KICAD9_3DMODEL_DIR}/Connector_IDC.3dshapes/IDC-Header_2x03_P2.54mm_Horizontal.step"
 			(offset
 				(xyz 0 0 0)
@@
 			)
 		)
-		(property "Value" "OPA365xxD"
+		(property "Value" "OPA365AIDR"
 			(at 0 3.4 0)
 			(layer "F.Fab")
@@
 		(layer "Edge.Cuts")
 	)
-	(gr_text "SWIR Wearable\nOptical Test\nV1.0 -2025-08\nE. Hazen"
+	(gr_text "NIR Wearable\nOptical Test\nV1.0 -2025-08\nE. Hazen"
 		(at 127.889 68.072 0)
 		(layer "F.SilkS")

Commit message: V1.0 as built
Parts:
- added D4: LED, LED_SMD:LED_0805_2012Metric_Pad1.15x1.40mm_HandSolder, F.Cu at (144.5, 102.7)
- added R11: 1.5k, Resistor_SMD:R_0805_2012Metric_Pad1.20x1.40mm_HandSolder, F.Cu at (140.0, 102.7)
- J1: footprint my_ScrewTerminal:TerminalBlock_TE_2POS_P5mm -> TerminalBlock:TerminalBlock_MaiXu_MX126-5.0-02P_1x02_P5.00mm
Connections:
- U7 pad 1: unconnected-(U7-PD3-Pad1) -> /GP_LED2
- U7 pad 14: unconnected-(U7-PB2-Pad14) -> /SS/DONT_USE
Routing:
- net /GP_LED2: track 0.00 -> 22.1 mm, vias 0 -> 2
- net Net-(D4-A): track 0.00 -> 7.11 mm
- net GND: track 42.5 -> 43.9 mm, vias 23 -> 24

Commit message: more tests
Parts:
- added N1: Optical_PCB, optical_pcb_model:optical_pcb, F.Cu at (116.8, 57.1)
Changed lines of the file:
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@@
 		)
 	)
+	(footprint "optical_pcb_model:optical_pcb"
+		(layer "F.Cu")
+		(at 116.84 57.15)
+		(property "Reference" "N1"
+			(at 0 -0.5 0)
+			(unlocked yes)
+			(layer "F.SilkS")
+			(effects
+				(font
+					(size 1 1)
+					(thickness 0.1)
+				)
+			)
+		)
+		(property "Value" "Optical_PCB"
+			(at 0 1 0)
+			(unlocked yes)
+			(layer "F.Fab")
+			(effects
+				(font
+					(size 1 1)
+					(thickness 0.15)
+				)
+			)
+		)
+		(property "Datasheet" "~"
+			(at 0 0 0)
+			(unlocked yes)
+			(layer "F.Fab")
+			(hide yes)
+			(effects
+				(font
+					(size 1 1)
+					(thickness 0.15)
+				)
+			)
+		)
+		(property "Description" "Housing"
+			(at 0 0 0)
+			(unlocked yes)
+			(layer "F.Fab")
+			(hide yes)
+			(effects
+				(font
+					(size 1 1)
+					(thickness 0.15)
+				)
+			)
+		)
+		(property ki_fp_filters "Enclosure* Housing*")
+		(sheetname "/")
+		(sheetfile "led-photodiode-avr.kicad_sch")
+		(attr smd)
+		(fp_rect
+			(start 0 0)
+			(end 68.58 80.01)
+			(stroke
+				(width 0.1)
+				(type default)
+			)
+			(fill no)
+			(layer "F.SilkS")
+		)
+		(fp_rect
+			(start 0 0)
+			(end 68.58 80.01)
+			(stroke
+				(width 0.1)
+				(type default)
+			)
+			(fill no)
+			(layer "User.2")
+		)
+		(fp_text user "${REFERENCE}"
+			(at 0 2.5 0)
+			(unlocked yes)
+			(layer "F.Fab")
+			(effects
+				(font
+					(size 1 1)
+					(thickness 0.15)
+				)
+			)
+		)
+		(pad "1" thru_hole circle
+			(at 5.08 5.08)
+			(size 4.572 4.572)
+			(drill 3.175)
+			(layers "*.Cu" "*.Mask")
+			(remove_unused_layers no)
+		)
+		(embedded_fonts no)
+		(model "${KIPRJMOD}/models/optical-carrier.wrl"
+			(offset
+				(xyz -169.545 55.88 12.065)
+			)
+			(scale
+				(xyz 0.392 0.392 0.392)
+			)
+			(rotate
+				(xyz -0 -0 -0)
+			)
+		)
+	)
 	(footprint "LED_SMD:LED_0805_2012Metric_Pad1.15x1.40mm_HandSolder"
 		(layer "F.Cu")
@@
 			(roundrect_rratio 0.25)
 			(net 6 "VCC")
-			(pinfunction "REF_SEL")
+			(pinfunction "CA1")
 			(pintype "passive")
 		)
@@
 		(layer "User.2")
 		(pts
+			(xy 116.84 57.15) (xy 121.92 62.23)
+		)
+		(height -6.604)
+		(orientation 0)
+		(format
+			(prefix "")
+			(suffix "")
+			(units 3)
+			(units_format 0)
+			(precision 4)
+			(suppress_zeroes yes)
+		)
+		(style
+			(thickness 0.1)
+			(arrow_length 1.27)
+			(text_position_mode 0)
+			(arrow_direction outward)
+			(extension_height 0.58642)
+			(extension_offset 0.5)
+			(keep_text_aligned yes)
+		)
+		(gr_text "0.2"
+			(at 119.38 49.396 0)
+			(layer "User.2")
+			(effects
+				(font
+					(size 1 1)
+					(thickness 0.15)
+				)
+			)
+		)
+	)
+	(dimension
+		(type orthogonal)
+		(layer "User.2")
+		(pts
 			(xy 180.34 62.23) (xy 180.34 132.08)
 		)
@@
 			(layer "User.2")
 			(effects
+				(font
+					(size 1 1)
+					(thickness 0.15)
+				)
+			)
+		)
+	)
+	(dimension
+		(type orthogonal)
+		(layer "User.2")
+		(pts
+			(xy 116.84 57.15) (xy 121.92 62.23)
+		)
+		(height -3.429)
+		(orientation 1)
+		(format
+			(prefix "")
+			(suffix "")
+			(units 3)
+			(units_format 0)
+			(precision 4)
+			(suppress_zeroes yes)
+		)
+		(style
+			(thickness 0.1)
+			(arrow_length 1.27)
+			(text_position_mode 0)
+			(arrow_direction outward)
+			(extension_height 0.58642)
+			(extension_offset 0.5)
+			(keep_text_aligned yes)
+		)
+		(gr_text "0.2"
+			(at 112.261 59.69 90)
+			(layer "User.2")
+			(effects

Commit message: working on main board changes, schem done
Parts:
- added C24: C, Capacitor_SMD:C_0805_2012Metric_Pad1.18x1.45mm_HandSolder, F.Cu at (210.2, 81.2)
- added C25: C, Capacitor_SMD:C_0805_2012Metric_Pad1.18x1.45mm_HandSolder, F.Cu at (210.2, 84.2)
- added C26: 0.1uF, Capacitor_SMD:C_0805_2012Metric_Pad1.18x1.45mm_HandSolder, F.Cu at (195.6, 66.5)
- added Q5: TTC1949, Package_TO_SOT_SMD:SC-59, F.Cu at (195.3, 82.2)
- added Q6: TTC1949, Package_TO_SOT_SMD:SC-59, F.Cu at (195.3, 87.1)
- added Q7: TTC1949, Package_TO_SOT_SMD:SC-59, F.Cu at (195.3, 91.9)
- added Q8: TTC1949, Package_TO_SOT_SMD:SC-59, F.Cu at (195.3, 96.7)
- added R12: 10k, Resistor_SMD:R_0805_2012Metric_Pad1.20x1.40mm_HandSolder, F.Cu at (200.6, 70.8)
- added TP1: TP, TestPoint:TestPoint_Pad_D1.0mm, F.Cu at (201.8, 81.8)
- added TP2: TP, TestPoint:TestPoint_Pad_D1.0mm, F.Cu at (201.8, 85.8)
- added TP3: TP, TestPoint:TestPoint_Pad_D1.0mm, F.Cu at (201.8, 89.8)
- added TP4: TP, TestPoint:TestPoint_Pad_D1.0mm, F.Cu at (201.8, 93.9)
- added TP5: TP, TestPoint:TestPoint_Pad_D1.0mm, F.Cu at (205.8, 81.8)
- added TP6: TP, TestPoint:TestPoint_Pad_D1.0mm, F.Cu at (205.8, 85.8)
- added TP7: TP, TestPoint:TestPoint_Pad_D1.0mm, F.Cu at (205.8, 89.8)
- added U11: MCP3221, Package_TO_SOT_SMD:SOT-23-5, F.Cu at (195.5, 71.0)
Connections:
- J2 pad 1: /LED_driver/LED_3 -> /LED_driver/LED_1
- J2 pad 10: unconnected-(J2-Pin_10-Pad10) -> +5VA
- J2 pad 11: /LED_driver/LED_K -> /LED_driver/LED_6
- J2 pad 13: unconnected-(J2-Pin_13-Pad13) -> /LED_driver/LED_7
- J2 pad 15: unconnected-(J2-Pin_15-Pad15) -> /LED_driver/LED_8
- J2 pad 3: /LED_driver/LED_K -> /LED_driver/LED_2
- J2 pad 5: /LED_driver/LED_2 -> /LED_driver/LED_3
- J2 pad 6: unconnected-(J2-Pin_6-Pad6) -> /TSENSE
- J2 pad 7: /LED_driver/LED_K -> /LED_driver/LED_4
- J2 pad 8: unconnected-(J2-Pin_8-Pad8) -> +5VA
- J2 pad 9: /LED_driver/LED_1 -> /LED_driver/LED_5
- Q1 pad 2: /LED_driver/LED_1 -> Net-(Q1-E)
- Q1 pad 3: +5VA -> /LED_driver/LED_1
- Q2 pad 2: /LED_driver/LED_2 -> Net-(Q1-E)
- Q2 pad 3: +5VA -> /LED_driver/LED_2
- Q3 pad 2: /LED_driver/LED_3 -> Net-(Q1-E)
- Q3 pad 3: +5VA -> /LED_driver/LED_3
- Q4 pad 2: /LED_driver/LED_4 -> Net-(Q1-E)
- Q4 pad 3: +5VA -> /LED_driver/LED_4
- R6 pad 1: /LED_driver/LED_K -> Net-(Q1-E)
- R7 pad 2: /LED_driver/LED_K -> Net-(Q1-E)
- U5 pad 23: unconnected-(U5-CAP2A-Pad23) -> Net-(C24-Pad2)
- U5 pad 24: Net-(C20-Pad1) -> Net-(C24-Pad1)
- U5 pad 26: unconnected-(U5-CAP2B-Pad26) -> Net-(C20-Pad1)
- U5 pad 3: unconnected-(U5-CAP1B-Pad3) -> Net-(C25-Pad2)
- U5 pad 4: Net-(C19-Pad2) -> Net-(C25-Pad1)
- U5 pad 5: Net-(C19-Pad1) -> Net-(C19-Pad2)
- U5 pad 6: unconnected-(U5-CAP1A-Pad6) -> Net-(C19-Pad1)
- U6 pad 5: unconnected-(U6-4-Pad5) -> Net-(Q5-B)
- U6 pad 6: unconnected-(U6-5-Pad6) -> Net-(Q6-B)
- U6 pad 7: unconnected-(U6-6-Pad7) -> Net-(Q7-B)
- U6 pad 8: unconnected-(U6-7-Pad8) -> Net-(Q8-B)
Routing:
- net /LED_driver/LED_K: track 27.3 -> 0.00 mm, vias 1 -> 0
- net (no net): track 0.00 -> 27.3 mm
- net /LED_driver/LED_1: track 10.2 -> 21.9 mm, vias 0 -> 1
- net /LED_driver/LED_2: track 10.3 -> 1.27 mm, vias 0 -> 1
- net +5VA: track 29.6 -> 24.4 mm, vias 15 -> 11
- net /LED_driver/LED_4: track 0.00 -> 1.40 mm, vias 0 -> 1
- net /LED_driver/LED_3: track 10.6 -> 11.7 mm, vias 0 -> 1
- net Net-(Q1-E): vias 0 -> 1
