File: KiCAD/led-photodiode-avr/LED_driver.kicad_sch (KiCad schematic)
At the start: 18 parts, among them Q1 TTC1949, Q2 TTC1949, Q3 TTC1949, Q4 TTC1949, U6 LTC1380, U8 OPA365xxD, U9 LTC2631

Commit message: working on BOM
Parts:
- C15: DigikeyNumber 1276-2048-1-ND -> 1276-1123-1-ND; ManufacturerNumber CL10B334KO8NNNC -> CL21B334KBFNNNE
- C16, C22: DigikeyNumber 1276-1005-1-ND -> 478-KGM21NR71H104KTCT-ND; ManufacturerNumber CL10B104KO8NNNC -> KGM21NR71H104KT
- C17: DigikeyNumber (none) -> 399-C0805C121J3GACTUCT-ND; ManufacturerNumber (none) -> C0805C121J3GACTU
- C18: DigikeyNumber (none) -> 478-KGM21NR71H104KTCT-ND; ManufacturerNumber (none) -> KGM21NR71H104KT
- C21: DigikeyNumber (none) -> 399-C0805C102J5GACTUCT-ND; ManufacturerNumber (none) -> C0805C102J5GACTU
Changed lines of the file:
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@@
 			)
 		)
-		(property "DigikeyNumber" ""
+		(property "DigikeyNumber" "478-KGM21NR71H104KTCT-ND"
 			(at 118.11 45.72 0)
 			(effects
@@
 			)
 		)
-		(property "ManufacturerNumber" ""
+		(property "ManufacturerNumber" "KGM21NR71H104KT"
 			(at 118.11 45.72 0)
 			(effects
@@
 			)
 		)
-		(property "DigikeyNumber" ""
+		(property "DigikeyNumber" "399-C0805C102J5GACTUCT-ND"
 			(at 90.17 59.69 0)
 			(effects
@@
 			)
 		)
-		(property "ManufacturerNumber" ""
+		(property "ManufacturerNumber" "C0805C102J5GACTU"
 			(at 90.17 59.69 0)
 			(effects
@@
 			)
 		)
-		(property "DigikeyNumber" "1276-1005-1-ND"
+		(property "DigikeyNumber" "478-KGM21NR71H104KTCT-ND"
 			(at 167.64 43.18 0)
 			(effects
@@
 			)
 		)
-		(property "ManufacturerNumber" "CL10B104KO8NNNC"
+		(property "ManufacturerNumber" "KGM21NR71H104KT"
 			(at 167.64 43.18 0)
 			(effects
@@
 			)
 		)
-		(property "DigikeyNumber" "1276-2048-1-ND"
+		(property "DigikeyNumber" "1276-1123-1-ND"
 			(at 26.67 59.69 0)
 			(effects
@@
 			)
 		)
-		(property "ManufacturerNumber" "CL10B334KO8NNNC"
+		(property "ManufacturerNumber" "CL21B334KBFNNNE"
 			(at 26.67 59.69 0)
 			(effects
@@
 			)
 		)
-		(property "DigikeyNumber" ""
+		(property "DigikeyNumber" "399-C0805C121J3GACTUCT-ND"
 			(at 110.49 78.74 0)
 			(effects
@@
 			)
 		)
-		(property "ManufacturerNumber" ""
+		(property "ManufacturerNumber" "C0805C121J3GACTU"
 			(at 110.49 78.74 0)
 			(effects
@@
 			)
 		)
-		(property "DigikeyNumber" "1276-1005-1-ND"
+		(property "DigikeyNumber" "478-KGM21NR71H104KTCT-ND"
 			(at 59.69 35.56 0)
 			(effects
@@
 			)
 		)
-		(property "ManufacturerNumber" "CL10B104KO8NNNC"
+		(property "ManufacturerNumber" "KGM21NR71H104KT"
 			(at 59.69 35.56 0)
 			(effects

Commit message: many schematic tweaks; add fields for BOM
Parts:
- R3, R5, R6: DigikeyNumber (none) -> 541-1.00KCCT-ND; ManufacturerNumber (none) -> CRCW08051K00FKEA
- R4: value 440 -> 442; DigikeyNumber (none) -> 311-442CRCT-ND; ManufacturerNumber (none) -> RC0805FR-07442RL
- R7: value 25 -> 24.9; DigikeyNumber (none) -> 541-CRCW120624R9FKEAHPCT-ND; ManufacturerNumber (none) -> CRCW120624R9FKEAHP
- U6: ManufacturerNumber (none) -> LTC1380CS#PBF
- U8: DigikeyNumber (none) -> 296-46162-1-ND; ManufacturerNumber (none) -> OPA365AIDR
Changed lines of the file:
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@@
 			)
 		)
-		(property "DigikeyNumber" ""
+		(property "DigikeyNumber" "541-1.00KCCT-ND"
 			(at 123.19 130.81 0)
 			(effects
@@
 			)
 		)
-		(property "ManufacturerNumber" ""
+		(property "ManufacturerNumber" "CRCW08051K00FKEA"
 			(at 123.19 130.81 0)
 			(effects
@@
 			)
 		)
-		(property "DigikeyNumber" ""
+		(property "DigikeyNumber" "541-1.00KCCT-ND"
 			(at 130.81 57.15 0)
 			(effects
@@
 			)
 		)
-		(property "ManufacturerNumber" ""
+		(property "ManufacturerNumber" "CRCW08051K00FKEA"
 			(at 130.81 57.15 0)
 			(effects
@@
 			)
 		)
-		(property "Value" "25"
+		(property "Value" "24.9"
 			(at 229.362 137.16 0)
 			(effects
@@
 			)
 		)
-		(property "DigikeyNumber" ""
+		(property "DigikeyNumber" "541-CRCW120624R9FKEAHPCT-ND"
 			(at 226.06 137.16 0)
 			(effects
@@
 			)
 		)
-		(property "ManufacturerNumber" ""
+		(property "ManufacturerNumber" "CRCW120624R9FKEAHP"
 			(at 226.06 137.16 0)
 			(effects
@@
 			)
 		)
+		(property "ManufacturerNumber" "LTC1380CS#PBF"
+			(at 147.32 57.15 0)
+			(effects
+				(font
+					(size 1.27 1.27)
+				)
+				(hide yes)
+			)
+		)
 		(pin "2"
 		)
@@
 			)
 		)
-		(property "Value" "440"
+		(property "Value" "442"
 			(at 83.5914 60.7568 90)
 			(effects
@@
 			)
 		)
-		(property "DigikeyNumber" ""
+		(property "DigikeyNumber" "311-442CRCT-ND"
 			(at 81.28 59.69 0)
 			(effects
@@
 			)
 		)
-		(property "ManufacturerNumber" ""
+		(property "ManufacturerNumber" "RC0805FR-07442RL"
 			(at 81.28 59.69 0)
 			(effects
@@
 			)
 		)
+		(property "DigikeyNumber" "296-46162-1-ND"
+			(at 113.03 57.15 0)
+			(effects
+				(font
+					(size 1.27 1.27)
+				)
+				(hide yes)
+			)
+		)
+		(property "ManufacturerNumber" "OPA365AIDR"
+			(at 113.03 57.15 0)
+			(effects
+				(font
+					(size 1.27 1.27)
+				)
+				(hide yes)
+			)
+		)
 		(pin "6"
 		)
@@
 			)
 		)
-		(property "DigikeyNumber" ""
+		(property "DigikeyNumber" "541-1.00KCCT-ND"
 			(at 74.93 54.61 0)
 			(effects
@@
 			)
 		)
-		(property "ManufacturerNumber" ""
+		(property "ManufacturerNumber" "CRCW08051K00FKEA"
 			(at 74.93 54.61 0)
 			(effects

Commit message: routing done
Connections:
- net Earth: no longer U6.11 (GND), U6.12 (A1), U6.13 (A0)
- net GND: now also U6.11 (GND), U6.12 (A1), U6.13 (A0)
- net LED_PWR_5V: no longer C16.1, U9.5 (VCC), U9.8 (REF_SEL)
- new net VCC: C16.1, U9.5 (VCC), U9.8 (REF_SEL)

Commit message: ready for review
Parts:
- U8: value OPA365xxD -> OPA365AIDR
Changed lines of the file:
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@@
 			)
 		)
-		(property "Value" "OPA365xxD"
+		(property "Value" "OPA365AIDR"
 			(at 118.364 64.77 0)
 			(effects

Commit message: readout working
Other:
- note added: "DAC range 0...4.095V I2C address = 0x44"
- note removed: "DAC range 0...4.095V"
Changed lines of the file:
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@@
 	(generator_version "9.0")
 	(paper "A4")
-	(text "DAC range 0...4.095V"
+	(text "DAC range 0...4.095V\nI2C address = 0x44"
 		(exclude_from_sim no)
-		(at 27.94 80.01 0)
+		(at 26.67 82.296 0)
 		(effects
 			(font

Commit message: starting on V2
Parts:
- added Q5, Q6, Q7, Q8: TTC1949, Package_TO_SOT_SMD:SC-59, symbol my_BJT:TTC1949
Connections:
- net LED_1: now also Q1.3 (C); no longer Q1.2 (E)
- net LED_2: now also Q2.3 (C); no longer Q2.2 (E)
- net LED_3: now also Q3.3 (C); no longer Q3.2 (E)
- net LED_4: now also Q4.3 (C); no longer Q4.2 (E)
- net at U6.5 (4): now also Q5.1 (B)
- net at U6.6 (5): now also Q6.1 (B)
- net at U6.7 (6): now also Q7.1 (B)
- net at U6.8 (7): now also Q8.1 (B)
- net LED_K: no longer names the net of R6.1, R7.2
- net LED_K: now also Q1.2 (E), Q2.2 (E), Q3.2 (E), Q4.2 (E), Q5.2 (E), Q6.2 (E), Q7.2 (E), Q8.2 (E)
- net LED_PWR_5V renamed LED_A
- net LED_A: no longer Q1.3 (C), Q2.3 (C), Q3.3 (C), Q4.3 (C)
- new net LED_5: Q5.3 (C)
- new net LED_6: Q6.3 (C)
- new net LED_7: Q7.3 (C)
- new net LED_8: Q8.3 (C)
Other:
- moved on the sheet: Q1, Q2, Q3, Q4, R6, R7

Commit message: Add op-amp buffer on temp sensor
Parts:
- renumbered C15 to C1, C16 to C3, C21 to C4, C18 to C5, C17 to C6, C22 to C7, Q7 to Q1, Q8 to Q2, Q5 to Q3, Q6 to Q4, Q4 to Q5, Q3 to Q6, Q2 to Q7, Q1 to Q8, R3 to R1, R4 to R2, R5 to R3, R6 to R8, R7 to R9, U9 to U2, U8 to U3, U6 to U5
Changed lines of the file:
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@@
 		(on_board yes)
 		(dnp no)
-		(property "Reference" "R6"
+		(property "Reference" "R8"
 			(at 120.65 147.066 90)
 			(effects
@@
 			(project "ddc112-shield"
 				(path "/e63e39d7-6ac0-4ffd-8aa3-1841a4541b55/85a88638-d0c9-4ca3-93c4-2444fc65b8fa"
-					(reference "R6")
+					(reference "R8")
 					(unit 1)
 				)
@@
 		(on_board yes)
 		(dnp no)
-		(property "Reference" "R5"
+		(property "Reference" "R3"
 			(at 130.81 62.357 90)
 			(effects
@@
 			(project "ddc112-shield"
 				(path "/e63e39d7-6ac0-4ffd-8aa3-1841a4541b55/85a88638-d0c9-4ca3-93c4-2444fc65b8fa"
-					(reference "R5")
+					(reference "R3")
 					(unit 1)
 				)
@@
 		(on_board yes)
 		(dnp no)
-		(property "Reference" "R7"
+		(property "Reference" "R9"
 			(at 229.362 151.384 0)
 			(effects
@@
 			(project "ddc112-shield"
 				(path "/e63e39d7-6ac0-4ffd-8aa3-1841a4541b55/85a88638-d0c9-4ca3-93c4-2444fc65b8fa"
-					(reference "R7")
+					(reference "R9")
 					(unit 1)
 				)
@@
 		(on_board yes)
 		(dnp no)
-		(property "Reference" "Q1"
+		(property "Reference" "Q8"
 			(at 229.6414 36.9316 0)
 			(effects
@@
 			(project "ddc112-shield"
 				(path "/e63e39d7-6ac0-4ffd-8aa3-1841a4541b55/85a88638-d0c9-4ca3-93c4-2444fc65b8fa"
-					(reference "Q1")
+					(reference "Q8")
 					(unit 1)
 				)
@@
 		(dnp no)
 		(fields_autoplaced yes)
-		(property "Reference" "U6"
+		(property "Reference" "U5"
 			(at 155.8133 45.72 0)
 			(effects
@@
 			(project ""
 				(path "/e63e39d7-6ac0-4ffd-8aa3-1841a4541b55/85a88638-d0c9-4ca3-93c4-2444fc65b8fa"
-					(reference "U6")
+					(reference "U5")
 					(unit 1)
 				)
@@
 		(on_board yes)
 		(dnp no)
-		(property "Reference" "Q3"
+		(property "Reference" "Q6"
 			(at 229.6414 64.8716 0)
 			(effects
@@
 			(project "ddc112-shield"
 				(path "/e63e39d7-6ac0-4ffd-8aa3-1841a4541b55/85a88638-d0c9-4ca3-93c4-2444fc65b8fa"
-					(reference "Q3")
+					(reference "Q6")
 					(unit 1)
 				)
@@
 		(on_board yes)
 		(dnp no)
-		(property "Reference" "Q6"
+		(property "Reference" "Q4"
 			(at 229.6414 106.7816 0)
 			(effects
@@
 			(project "led-photodiode-avr"
 				(path "/e63e39d7-6ac0-4ffd-8aa3-1841a4541b55/85a88638-d0c9-4ca3-93c4-2444fc65b8fa"
-					(reference "Q6")
+					(reference "Q4")
 					(unit 1)
 				)
@@
 		(on_board yes)
 		(dnp no)
-		(property "Reference" "R4"
+		(property "Reference" "R2"
 			(at 78.994 59.3598 90)
 			(effects
@@
 			(project "ddc112-shield"
 				(path "/e63e39d7-6ac0-4ffd-8aa3-1841a4541b55/85a88638-d0c9-4ca3-93c4-2444fc65b8fa"
-					(reference "R4")
+					(reference "R2")
 					(unit 1)
 				)
@@
 		(on_board yes)
 		(dnp no)
-		(property "Reference" "Q4"
+		(property "Reference" "Q5"
 			(at 229.6414 78.8416 0)
 			(effects
@@
 			(project "ddc112-shield"
 				(path "/e63e39d7-6ac0-4ffd-8aa3-1841a4541b55/85a88638-d0c9-4ca3-93c4-2444fc65b8fa"
-					(reference "Q4")
+					(reference "Q5")
 					(unit 1)
 				)
@@
 		(on_board yes)
 		(dnp no)
-		(property "Reference" "C18"
+		(property "Reference" "C5"
 			(at 112.014 45.466 0)
 			(effects
@@
 			(project "ddc112-shield"
 				(path "/e63e39d7-6ac0-4ffd-8aa3-1841a4541b55/85a88638-d0c9-4ca3-93c4-2444fc65b8fa"
-					(reference "C18")
+					(reference "C5")
 					(unit 1)
 				)
@@
 		(on_board yes)
 		(dnp no)
-		(property "Reference" "Q5"
+		(property "Reference" "Q3"
 			(at 229.6414 92.8116 0)
 			(effects
@@
 			(project "led-photodiode-avr"
 				(path "/e63e39d7-6ac0-4ffd-8aa3-1841a4541b55/85a88638-d0c9-4ca3-93c4-2444fc65b8fa"
-					(reference "Q5")
+					(reference "Q3")
 					(unit 1)
 				)
@@
 		(on_board yes)
 		(dnp no)
-		(property "Reference" "C21"
+		(property "Reference" "C4"
 			(at 92.71 58.4263 0)
 			(effects
@@
 			(project "ddc112-shield"
 				(path "/e63e39d7-6ac0-4ffd-8aa3-1841a4541b55/85a88638-d0c9-4ca3-93c4-2444fc65b8fa"
-					(reference "C21")
+					(reference "C4")
 					(unit 1)
 				)
@@
 		(on_board yes)
 		(dnp no)
-		(property "Reference" "U9"
+		(property "Reference" "U2"
 			(at 57.15 59.944 0)
 			(effects
@@
 			(project "ddc112-shield"
 				(path "/e63e39d7-6ac0-4ffd-8aa3-1841a4541b55/85a88638-d0c9-4ca3-93c4-2444fc65b8fa"
-					(reference "U9")
+					(reference "U2")
 					(unit 1)
 				)
@@
 		(on_board yes)
 		(dnp no)
-		(property "Reference" "C22"
+		(property "Reference" "C7"
 			(at 170.18 41.9163 0)
 			(effects
@@
 			(project "ddc112-shield"
 				(path "/e63e39d7-6ac0-4ffd-8aa3-1841a4541b55/85a88638-d0c9-4ca3-93c4-2444fc65b8fa"
-					(reference "C22")
+					(reference "C7")
 					(unit 1)
 				)
@@
 		(on_board yes)
 		(dnp no)
-		(property "Reference" "C15"
+		(property "Reference" "C1"
 			(at 24.13 58.4263 0)
 			(effects
@@
 			(project "ddc112-shield"
 				(path "/e63e39d7-6ac0-4ffd-8aa3-1841a4541b55/85a88638-d0c9-4ca3-93c4-2444fc65b8fa"
-					(reference "C15")
+					(reference "C1")
 					(unit 1)
 				)
@@
 		(on_board yes)
 		(dnp no)
-		(property "Reference" "C17"
+		(property "Reference" "C6"
 			(at 109.3216 75.819 90)
 			(effects
@@
 			(project "ddc112-shield"
 				(path "/e63e39d7-6ac0-4ffd-8aa3-1841a4541b55/85a88638-d0c9-4ca3-93c4-2444fc65b8fa"
-					(reference "C17")
+					(reference "C6")
 					(unit 1)
 				)
@@
 		(on_board yes)
 		(dnp no)
-		(property "Reference" "Q8"
+		(property "Reference" "Q2"
 			(at 229.6414 134.7216 0)
 			(effects
@@
 			(project "led-photodiode-avr"
 				(path "/e63e39d7-6ac0-4ffd-8aa3-1841a4541b55/85a88638-d0c9-4ca3-93c4-2444fc65b8fa"
-					(reference "Q8")
+					(reference "Q2")
 					(unit 1)
 				)
@@
 		(on_board yes)
 		(dnp no)
-		(property "Reference" "U8"
+		(property "Reference" "U3"
 			(at 114.3 62.23 0)
 			(effects
@@
 			(project ""
 				(path "/e63e39d7-6ac0-4ffd-8aa3-1841a4541b55/85a88638-d0c9-4ca3-93c4-2444fc65b8fa"
-					(reference "U8")
+					(reference "U3")
 					(unit 1)
 				)
@@
 		(on_board yes)
 		(dnp no)
-		(property "Reference" "Q2"
+		(property "Reference" "Q7"
 			(at 229.6414 50.9016 0)
 			(effects
@@
 			(project "ddc112-shield"
 				(path "/e63e39d7-6ac0-4ffd-8aa3-1841a4541b55/85a88638-d0c9-4ca3-93c4-2444fc65b8fa"
-					(reference "Q2")
+					(reference "Q7")
 					(unit 1)
 				)
@@
 		(on_board yes)
 		(dnp no)
-		(property "Reference" "R3"
+		(property "Reference" "R1"
 			(at 78.3844 52.6796 90)
 			(effects
@@
 			(project "ddc112-shield"
 				(path "/e63e39d7-6ac0-4ffd-8aa3-1841a4541b55/85a88638-d0c9-4ca3-93c4-2444fc65b8fa"
-					(reference "R3")
+					(reference "R1")
 					(unit 1)
 				)
@@
 		(on_board yes)
 		(dnp no)
-		(property "Reference" "C16"
+		(property "Reference" "C3"
 			(at 62.23 34.2963 0)
 			(effects
@@
 			(project "ddc112-shield"
 				(path "/e63e39d7-6ac0-4ffd-8aa3-1841a4541b55/85a88638-d0c9-4ca3-93c4-2444fc65b8fa"
-					(reference "C16")
+					(reference "C3")
 					(unit 1)
 				)
@@
 		(on_board yes)
 		(dnp no)
-		(property "Reference" "Q7"
+		(property "Reference" "Q1"
 			(at 229.6414 120.7516 0)
 			(effects
@@
 			(project "led-photodiode-avr"
 				(path "/e63e39d7-6ac0-4ffd-8aa3-1841a4541b55/85a88638-d0c9-4ca3-93c4-2444fc65b8fa"
-					(reference "Q7")
-					(unit 1)
-				)
+					(reference "Q1")
+					(unit 1)
+				)

Commit message: hopefully final Rev 2
Connections:
- net at Q8.1 (B): now also U5.6 (5); no longer U5.1 (0)
- net at U5.2 (1): now also Q3.1 (B); no longer Q7.1 (B)
- net at U5.3 (2): now also Q5.1 (B); no longer Q6.1 (B)
- net at U5.4 (3): now also Q6.1 (B); no longer Q5.1 (B)
- net at U5.5 (4): now also Q7.1 (B); no longer Q3.1 (B)
- net at Q4.1 (B): now also U5.1 (0); no longer U5.6 (5)
