File: KiCAD/optical-carrier/optical-carrier.kicad_pcb (KiCad board)
At the start: 2 copper layers, 68.6 x 80 mm, 9 parts, among them J1 Conn_02x08_Odd_Even

Commit message: V1.0 as built
Other:
- board text added: "NIR Wearable LED / Phototdiode test carrier V1.0 - 2025-08"
- board text removed: "SCOS Wearable LED / Phototdiode test carrier V1.0 - 2025-08"
Changed lines of the file:
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@@
 		(tenting front back)
 		(pcbplotparams
-			(layerselection 0x00000000_00000000_55555555_5755f5ff)
+			(layerselection 0x00000000_00000000_55555555_575555ff)
 			(plot_on_all_layers_selection 0x00000000_00000000_00000000_00000000)
 			(disableapertmacros no)
@@
 			(outputformat 1)
 			(mirror no)
-			(drillshape 1)
+			(drillshape 0)
 			(scaleselection 1)
-			(outputdirectory "")
+			(outputdirectory "gerber/")
 		)
 	)
@@
 		(layer "Edge.Cuts")
 	)
-	(gr_text "SCOS Wearable\nLED / Phototdiode test carrier\nV1.0 - 2025-08"
+	(gr_text "NIR Wearable\nLED / Phototdiode test carrier\nV1.0 - 2025-08"
 		(at 184.3024 75.3618 0)
 		(layer "F.SilkS")

Commit message: working on v2 layout
Parts:
- removed H1, H2, H3, H4: , 
- added D1: LED_GABR, my_LED:Marubeni, F.Cu at (212.2, 111.4)
- added D5: LED_GABR, my_LED:Marubeni, F.Cu at (187.2, 111.4)
- added JP1: Jumper_3_Bridged12, Connector_PinHeader_2.54mm:PinHeader_1x03_P2.54mm_Vertical, F.Cu at (192.2, 100.8)
- added TH1: Thermistor, Resistor_SMD:R_0603_1608Metric_Pad0.98x0.95mm_HandSolder, F.Cu at (233.4, 109.5)
- moved D6 0.09 mm to (200.3, 108.7)
- moved D2 0.08 mm to (215.3, 108.7)
- moved D3 0.06 mm to (190.3, 108.7)
- renumbered D3 to D2, D1 to D3, D2 to D6
Connections:
- net Net-(D1-K) renamed /LED2
- D2 pad 1: Net-(D3-K) -> /LED1
- D2 pad 2: Net-(D3-A) -> Net-(D1-A)
- D6 pad 1: Net-(D2-K) -> Net-(D6-K)
- D6 pad 2: Net-(D2-A) -> Net-(D1-A)
- J1 pad 1: Net-(D1-A) -> /LED1
- J1 pad 10: unconnected-(J1-Pin_10-Pad10) -> Net-(D1-A)
- J1 pad 11: Net-(D3-K) -> /LED6
- J1 pad 13: unconnected-(J1-Pin_13-Pad13) -> /LED7
- J1 pad 14: unconnected-(J1-Pin_14-Pad14) -> Net-(J1-Pin_14)
- J1 pad 15: unconnected-(J1-Pin_15-Pad15) -> /LED8
- J1 pad 5: Net-(D2-A) -> /LED3
- J1 pad 6: unconnected-(J1-Pin_6-Pad6) -> Net-(J1-Pin_6)
- J1 pad 7: Net-(D2-K) -> /LED4
- J1 pad 8: unconnected-(J1-Pin_8-Pad8) -> Net-(D1-A)
- J1 pad 9: Net-(D3-A) -> /LED5
Routing:
- net Net-(D1-A): track 59.7 -> 0.00 mm
- net /LED2: track 53.3 -> 0.00 mm
- net Net-(D2-A): track 40.5 -> 0.00 mm
- net Net-(D2-K): track 34.4 -> 0.00 mm
- net Net-(D3-A): track 22.4 -> 0.00 mm
- net Net-(D3-K): track 14.6 -> 0.00 mm
- net Net-(D4-K): track 6.11 -> 0.00 mm
- net Net-(D4-A): track 6.00 -> 0.00 mm

Commit message: routing done?
Parts:
- moved TH1 9.75 mm to (223.6, 109.5)
- moved JP1 5.74 mm to (194.2, 95.4)
- renumbered D5 to D1, D3 to D2, D2 to D3, D6 to D4, D1 to D5, D4 to D6
Connections:
- D1 pad 1: /LED7 -> /LED1
- D1 pad 4: /LED6 -> /LED3
- D3 pad 1: /LED1 -> /LED6
- D5 pad 1: /LED4 -> /LED5
- D5 pad 3: /LED5 -> /LED8
- D5 pad 4: /LED3 -> /LED7
- D6 pad 2: Net-(D4-A) -> Net-(D6-A)
- J1 pad 14: Net-(J1-Pin_14) -> Net-(D6-A)
- J1 pad 4: Net-(D4-A) -> Net-(D6-A)
- JP1 pad 2: /LED8 -> /LED4
- TH1 pad 2: Net-(J1-Pin_14) -> Net-(D6-A)
Routing:
- net /LED1: track 0.00 -> 80.7 mm
- net /LED2: track 0.00 -> 66.8 mm
- net /LED3: track 0.00 -> 64.7 mm
- net /LED5: track 0.00 -> 42.8 mm
- net /LED7: track 0.00 -> 35.2 mm
- net /LED6: track 0.00 -> 34.5 mm
- net /LED4: track 0.00 -> 31.8 mm
- net /LED8: track 0.00 -> 29.0 mm
- net Net-(D1-BK): track 0.00 -> 20.8 mm
- net Net-(D4-K): track 0.00 -> 13.7 mm
- net Net-(J1-Pin_6): track 0.00 -> 12.1 mm, vias 0 -> 1
- net Net-(D1-A): track 0.00 -> 6.59 mm, vias 0 -> 5
- net Net-(D6-K): track 0.00 -> 6.11 mm
- added copper zone on B.Cu, net Net-(D1-A)
- added copper zone on B.Cu, net Net-(D6-A)
- added copper zone on F.Cu, net Net-(D6-A)
- removed copper zone on B.Cu, net Net-(D4-A)
- removed copper zone on F.Cu, net Net-(D4-A)
Other:
- board text added: "NIR Wearable LED / Phototdiode test carrier V2.0 - 2025-10 ESH"
- board text removed: "NIR Wearable LED / Phototdiode test carrier V1.0 - 2025-08"

Commit message: update schem PDF, readmes
Parts:
- added H1: MountingHole, MountingHole:MountingHole_4.3mm_M4_DIN965, F.Cu at (175.3, 61.0)
- added H2: MountingHole, MountingHole:MountingHole_4.3mm_M4_DIN965, F.Cu at (233.7, 61.0)
- added H3: MountingHole, MountingHole:MountingHole_4.3mm_M4_DIN965, F.Cu at (233.7, 130.8)
- added H4: MountingHole, MountingHole:MountingHole_4.3mm_M4_DIN965, F.Cu at (175.3, 130.8)

Commit message: hopefully final Rev 2
Parts:
- D1, D5: value LED_GABR -> Marubeni_LED
- TH1: value Thermistor -> 10K NTC B2585=3435K
Connections:
- D1 pad 1: /LED1 -> Net-(D1-A)
- D1 pad 2: Net-(D1-A) -> /LED1
- D5 pad 1: /LED5 -> Net-(D1-A)
- D5 pad 2: Net-(D1-A) -> /LED5
Routing:
- net /LED1: track 80.7 -> 81.3 mm
- net /LED5: track 42.8 -> 43.4 mm
